Commit message: update stable v1 env

File: source/ext_template/data/Robots/Panda/reddog_20250221/reddog_20250221/urdf/reddog_20250221.urdf (robot description, URDF)
Before this commit: robot reddog_20250221, 17 links, 16 joints
Joints:
- removed joint fl_ft
- removed joint fl_hx
- removed joint fl_hy
- removed joint fl_kn
- removed joint fr_ft
- removed joint fr_hx
- removed joint fr_hy
- removed joint fr_kn
- removed joint hl_ft
- removed joint hl_hx
- removed joint hl_hy
- removed joint hl_kn
- removed joint hr_ft
- removed joint hr_hx
- removed joint hr_hy
- removed joint hr_kn
- added joint FL_calf_joint: type revolute, parent FL_thigh, child FL_calf, origin xyz=0 0.0409852014855581 -0.130000000000001 rpy=0 0 0, axis 0 1 0, limit lower=-2.0 upper=0.0 effort=0.0 velocity=0.0
- added joint FL_foot_joint: type fixed, parent FL_calf, child FL_foot, origin xyz=0 0 -0.13 rpy=0 0 0, axis 0 1 0
- added joint FL_hip_joint: type revolute, parent base, child FL_hip, origin xyz=0.127999974999998 0.055 0 rpy=0 0 0, axis 1 0 0, limit lower=-0.3 upper=0.57 effort=0.0 velocity=0.0
- added joint FL_thigh_joint: type revolute, parent FL_hip, child FL_thigh, origin xyz=0.038500025 0.0375 0 rpy=0 0 0, axis 0 1 0, limit lower=0.0 upper=2.0 effort=0.0 velocity=0.0
- added joint FR_calf_joint: type revolute, parent FR_thigh, child FR_calf, origin xyz=0 -0.0409852014855582 -0.130000000000001 rpy=0 0 0, axis 0 1 0, limit lower=-2.0 upper=0.0 effort=0.0 velocity=0.0
- added joint FR_foot_joint: type fixed, parent FR_calf, child FR_foot, origin xyz=0 0 -0.13 rpy=0 0 0, axis 0 1 0
- added joint FR_hip_joint: type revolute, parent base, child FR_hip, origin xyz=0.127999974999998 -0.055 0 rpy=0 0 0, axis 1 0 0, limit lower=-0.57 upper=0.3 effort=0.0 velocity=0.0
- added joint FR_thigh_joint: type revolute, parent FR_hip, child FR_thigh, origin xyz=0.0385000250000002 -0.0374999999999999 0 rpy=0 0 0, axis 0 1 0, limit lower=0.0 upper=2.0 effort=0.0 velocity=0.0
- added joint RL_calf_joint: type revolute, parent RL_thigh, child RL_calf, origin xyz=0 0.0409852014855523 -0.130000000000005 rpy=0 0 0, axis 0 1 0, limit lower=0.0 upper=2.0 effort=0.0 velocity=0.0
- added joint RL_foot_joint: type fixed, parent RL_calf, child RL_foot, origin xyz=0 0 -0.130000000000004 rpy=0 0 0, axis 0 1 0
- added joint RL_hip_joint: type revolute, parent base, child RL_hip, origin xyz=-0.127999974999999 0.054999999999999 0 rpy=0 0 0, axis 1 0 0, limit lower=-0.3 upper=0.57 effort=0.0 velocity=0.0
- added joint RL_thigh_joint: type revolute, parent RL_hip, child RL_thigh, origin xyz=-0.0385000249999999 0.0374999999999952 0 rpy=0 0 0, axis 0 1 0, limit lower=-2.0 upper=0.0 effort=0.0 velocity=0.0
- added joint RR_calf_joint: type revolute, parent RR_thigh, child RR_calf, origin xyz=0 -0.040985201485548 -0.130000000000005 rpy=0 0 0, axis 0 1 0, limit lower=0.0 upper=2.0 effort=0.0 velocity=0.0
- added joint RR_foot_joint: type fixed, parent RR_calf, child RR_foot, origin xyz=0 0 -0.130000000000004 rpy=0 0 0, axis 0 1 0
- added joint RR_hip_joint: type revolute, parent base, child RR_hip, origin xyz=-0.127999975000002 -0.055 0 rpy=0 0 0, axis 1 0 0, limit lower=-0.57 upper=0.3 effort=0.0 velocity=0.0
- added joint RR_thigh_joint: type revolute, parent RR_hip, child RR_thigh, origin xyz=-0.0385000250000012 -0.0374999999999921 0 rpy=0 0 0, axis 0 1 0, limit lower=-2.0 upper=0.0 effort=0.0 velocity=0.0
